File: hw/protecao_entrada.kicad_sch (KiCad schematic)
At the start: 5 parts, among them Q1 AO3407A (Rds_on=28mOhm, -20V,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

Commit message: update(docs): atualiza protecoes-entrada e esquemático
Other:
- title: Micromouse PI1 - Malha de Protecao de Entrada (Issue #200) -> Micromouse PI1 - Malha de Protecao de Entrada
Changed lines of the file:
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@@
 	(paper "A4")
 	(title_block
-		(title "Micromouse PI1 - Malha de Protecao de Entrada (Issue #200)")
+		(title "Micromouse PI1 - Malha de Protecao de Entrada")
 		(date "2026-10-17")
 		(rev "1.0")
